File: usb to uart/usb to uart.kicad_pcb (KiCad board)
At the start: 2 copper layers, 39.5 x 14.5 mm, 22 parts, among them J1 USB_C_Receptacle_USB2.0_16P, J2 Conn_01x05, U1 CP2102N-Axx-xQFN28

Commit message: updated files
Parts:
- added REF**: WEEE-Logo_4.2x6mm_SilkScreen, Symbol:WEEE-Logo_4.2x6mm_SilkScreen, F.Cu at (120.2, 88.8)
Connections:
- U1 pad 4: /USB_DM -> /USB_DP
- U1 pad 5: /USB_DP -> /USB_DM
Routing:
- net Net-(U1-VDD): track 2.51 -> 22.2 mm, vias 0 -> 2
- net GND: track 0.00 -> 10.1 mm, vias 84 -> 88
- net Net-(J1-CC2): track 15.7 -> 12.7 mm
- net /UART_RX: track 31.3 -> 28.8 mm, vias 0 -> 2
- net Net-(D1-I/O2-Pad3): track 20.7 -> 18.7 mm, vias 0 -> 2
- net /UART_TX: track 24.9 -> 23.2 mm
- net /USB_DM: track 15.1 -> 13.8 mm
- net /USB_DP: track 9.18 -> 8.35 mm
- net /VBUS: track 41.3 -> 41.6 mm, vias 0 -> 2
- net Net-(J1-CC1): vias 0 -> 2
- added copper zone on B.Cu, net GND
Other:
- board text added: "GND"
- board text added: "RX"
- board text added: "TX"
- board text added: "VCC"
