File: usb to uart/usb to uart.kicad_sch (KiCad schematic)
At the start: 22 parts, among them J1 USB_C_Receptacle_USB2.0_16P, J2 Conn_01x05, U1 CP2102N-Axx-xQFN28

Commit message: updated files
Changed lines of the file:
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@@
 	(wire
 		(pts
-			(xy 251.46 102.87) (xy 260.35 102.87)
+			(xy 247.65 102.87) (xy 260.35 102.87)
 		)
 		(stroke
@@
 		(pts
 			(xy 223.52 60.96) (xy 223.52 49.53)
-		)
-		(stroke
-			(width 0)
-			(type default)
-		)
-	)
-	(wire
-		(pts
-			(xy 251.46 100.33) (xy 251.46 102.87)
 		)
 		(stroke
@@
 	(symbol
 		(lib_id "power:GND")
-		(at 251.46 100.33 180)
+		(at 247.65 102.87 270)
 		(unit 1)
 		(exclude_from_sim no)
@@
 		(fields_autoplaced yes)
 		(property "Reference" "#PWR09"
-			(at 251.46 93.98 0)
+			(at 241.3 102.87 0)
 			(effects
 				(font
@@
 		)
 		(property "Value" "GND"
-			(at 251.46 95.25 0)
+			(at 243.84 102.8699 90)
 			(effects
 				(font
 					(size 1.27 1.27)
 				)
+				(justify right)
 			)
 		)
 		(property "Footprint" ""
-			(at 251.46 100.33 0)
+			(at 247.65 102.87 0)
 			(effects
 				(font
@@
 		)
 		(property "Datasheet" ""
-			(at 251.46 100.33 0)
+			(at 247.65 102.87 0)
 			(effects
 				(font
@@
 		)
 		(property "Description" "Power symbol creates a global label with name \"GND\" , ground"
-			(at 251.46 100.33 0)
+			(at 247.65 102.87 0)
 			(effects
 				(font
